Commit message: body redesign and ros2 controller setup

File: ros2_ws/src/ejison/model/parameters.xacro (robot description, xacro)
@@ -14,4 +14,7 @@
         <color rgba="0.5 0.3 0 1" />
     </material>
+    <material name="yellow">
+        <color rgba="1 1 0 1" />
+    </material>
     <!-- Default Origin -->
     <xacro:macro name="default_origin">
@@ -21,6 +24,6 @@
     <xacro:property name="density" value="1200" />
     <!-- Base Link -->
-    <xacro:property name="body_length" value="0.26" />
-    <xacro:property name="body_breadth" value="0.205" />
+    <xacro:property name="body_length" value="0.205" />
+    <xacro:property name="body_breadth" value="0.18" />
     <xacro:property name="body_height" value="0.005" />
     <xacro:property name="body_mass" value="${density*body_length*body_breadth*body_height}" />
@@ -28,9 +31,14 @@
     <xacro:property name="wheel_radius" value="0.0325" />
     <xacro:property name="wheel_length" value="0.025" />
-    <xacro:property name="wheel_mass" value="${pi*wheel_radius*wheel_radius*wheel_length}" />
+    <xacro:property name="wheel_mass" value="${density*pi*wheel_radius*wheel_radius*wheel_length}" />
     <!-- Caster Wheel -->
     <xacro:property name="caster_wheel_radius" value="0.01625" />
     <xacro:property name="caster_wheel_mass"
         value="${(4.0/3.0)*pi*caster_wheel_radius*caster_wheel_radius*caster_wheel_radius}" />
+    <!-- Battery -->
+    <xacro:property name="battery_length" value="0.15" />
+    <xacro:property name="battery_breadth" value="0.07" />
+    <xacro:property name="battery_height" value="0.02" />
+    <xacro:property name="battery_mass" value="0.25" />
     <!-- Camera -->
     <xacro:property name="camera_length" value="0.07" />

File: ros2_ws/src/ejison/model/robot_core.xacro (robot description, xacro)
@@ -67,5 +67,5 @@
         <parent link="base_link" />
         <child link="left_wheel_link" />
-        <origin xyz="-0.08 0.115 0" rpy="0 0 0" />
+        <origin xyz="-0.08 ${0.09+wheel_length/2} 0" rpy="0 0 0" />
         <axis xyz="0 1 0" />
     </joint>
@@ -76,5 +76,5 @@
         <parent link="base_link" />
         <child link="right_wheel_link" />
-        <origin xyz="-0.08 -0.115 0" rpy="0 0 0" />
+        <origin xyz="-0.08 -${0.09+wheel_length/2} 0" rpy="0 0 0" />
         <axis xyz="0 1 0" />
     </joint>
@@ -110,4 +110,38 @@
         <origin xyz="0.08 0 -0.01625" rpy="0 0 0" />
     </joint>
+    <!-- Battery -->
+    <link name="battery_link">
+        <visual>
+            <geometry>
+                <box size="${battery_length} ${battery_breadth} ${battery_height}" />
+            </geometry>
+            <origin xyz="0 0 0" rpy="0 0 1.57" />
+            <material name="yellow" />
+        </visual>
+        <collision>
+            <geometry>
+                <box size="${battery_length} ${battery_breadth} ${battery_height}" />
+            </geometry>
+            <origin xyz="0 0 0" rpy="0 0 1.57" />
+        </collision>
+        <inertial>
+            <mass value="${battery_mass}" />
+            <xacro:default_origin />
+            <inertia
+                ixx="${(1.0/12.0)*battery_mass*(battery_breadth*battery_breadth + battery_height*battery_height)}"
+                iyy="${(1.0/12.0)*battery_mass*(battery_length*battery_length + battery_height*battery_height)}"
+                izz="${(1.0/12.0)*battery_mass*(battery_length*battery_length + battery_breadth*battery_breadth)}"
+                ixy="0.0"
+                ixz="0.0"
+                iyz="0.0" />
+        </inertial>
+    </link>
+    <!-- Battery Joint -->
+    <joint name="battery_joint" type="fixed">
+        <parent link="base_link" />
+        <child link="battery_link" />
+        <origin xyz="${body_length/2-0.01-battery_breadth/2} 0 ${body_height+battery_height/2}"
+            rpy="0 0 0" />
+    </joint>
     <!-- Camera -->
     <link name="camera_link">
@@ -137,7 +171,7 @@
     <!-- Camera Joint -->
     <joint name="base_camera_joint" type="fixed">
-        <parent link="base_link" />
+        <parent link="battery_link" />
         <child link="camera_link" />
-        <origin xyz="0.1 0 0.0125" rpy="0 0 0" />
+        <origin xyz="0 0 ${battery_height/2+camera_height/2}" rpy="0 0 0" />
     </joint>
     <!-- Camera Lens -->
@@ -161,6 +195,8 @@
             <inertia
                 ixx="${(1.0/2.0)*camera_lens_mass*camera_lens_radius*camera_lens_radius}"
-                iyy="${(1.0/12.0)*camera_lens_mass*(3*camera_lens_radius*camera_lens_radius + camera_lens_length*camera_lens_length)}"
-                izz="${(1.0/12.0)*camera_lens_mass*(3*camera_lens_radius*camera_lens_radius + camera_lens_length*camera_lens_length)}"
+                iyy="${(1.0/12.0)*camera_lens_mass*(3*camera_lens_radius*camera_lens_radius +
+    camera_lens_length*camera_lens_length)}"
+                izz="${(1.0/12.0)*camera_lens_mass*(3*camera_lens_radius*camera_lens_radius +
+    camera_lens_length*camera_lens_length)}"
                 ixy="0.0" ixz="0.0" iyz="0.0" />
         </inertial>
